Commit message: First commit: Cartographer and Gazebo setup complete

File: install/fishbot_description/share/fishbot_description/urdf/urdf/fishbot_gazebo.urdf (robot description, URDF)
Before this commit: robot fishbot, 7 links, 6 joints
Links:
- added link ultrasonic_sensor_link
Joints:
- added joint ultrasonic_sensor_joint: type fixed, parent base_link, child ultrasonic_sensor_link, origin xyz=0.07 0.0 0.076 rpy=0 0 0
